Commit message: change coordinate

File: src/tactile_raw_point_publisher/urdf/Sensor_holer_URDF.urdf (robot description, URDF)
Before this commit: robot Sensor_holer, 3 links, 2 joints
Links:
- link sensor_1_link: mass 0 -> 0.0062307
- link sensor_3_link: mass 0.00623069775844809 -> 0.0062307
- link sensor_base: mass 0.144120684918715 -> 0.14412
Joints:
- joint sensor_1_link_joint: axis 0 0 0 -> 1 0 0; origin xyz=-0.0011986 0.002024 0.204 rpy=1.5708 0 -2.5629 -> xyz=-0.0020191 0.0032797 0.20148 rpy=-1.6223 0 -2.5629
- joint sensor_3_link_joint: origin xyz=0.0011986 -0.002024 0.204 rpy=1.5708 0 0.57871 -> xyz=0.0020191 -0.0032797 0.20148 rpy=-1.6223 0 0.57871
