Commit message: update coord

File: src/tactile_raw_point_publisher/urdf/Sensor_holer_nc.urdf (robot description, URDF)
Before this commit: robot Sensor_holer_nc, 3 links, 2 joints
Joints:
- joint sensor_1_link_joint: axis 1 0 0 -> 0 0 0; origin xyz=-0.0020191 0.0032797 0.20148 rpy=-1.6223 0 -2.5629 -> xyz=-0.0020191 0.0032797 0.20148 rpy=1.5193 0 -2.5629
- joint sensor_3_link_joint: origin xyz=0.0020191 -0.0032797 0.20148 rpy=-1.6223 0 0.57871 -> xyz=0.0020191 -0.0032797 0.20148 rpy=1.5193 0 0.57871
